Commit message: update urdf

File: files/BRUCE_V1.4_simplified.urdf (robot description, URDF)
Before this commit: robot BRUCE_V1.4_DUMMY_Sim_simplified, 17 links, 16 joints
Links:
- removed link ankle_pitch_l
- removed link ankle_pitch_r
- removed link elbow_pitch_l
- removed link elbow_pitch_r
- removed link hip_pitch_l
- removed link hip_pitch_r
- removed link hip_roll_l
- removed link hip_roll_r
- removed link hip_yaw_l
- removed link hip_yaw_r
- removed link knee_pitch_l
- removed link knee_pitch_r
- removed link shoulder_pitch_l
- removed link shoulder_pitch_r
- removed link shoulder_roll_l
- removed link shoulder_roll_r
- added link ankle_pitch_link_l, mass 0.027482910; collision mesh filename=package://BRUCE_V1.4_simplified/meshes/ankle_pitch_link_l.S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; visual mesh filename=package://BRUCE_V1.4_simplified/meshes/ankle_pitch_link_l.S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
- added link ankle_pitch_link_r, mass 0.027626470; collision mesh filename=package://BRUCE_V1.4_simplified/meshes/ankle_pitch_link_r.S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; visual mesh filename=package://BRUCE_V1.4_simplified/meshes/ankle_pitch_link_r.S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
- added link elbow_pitch_link_l, mass 0.052440370; collision mesh filename=package://BRUCE_V1.4_simplified/meshes/elbow_pitch_link_l.S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; visual mesh filename=package://BRUCE_V1.4_simplified/meshes/elbow_pitch_link_l.S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
- added link elbow_pitch_link_r, mass 0.052440370; collision mesh filename=package://BRUCE_V1.4_simplified/meshes/elbow_pitch_link_r.S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; visual mesh filename=package://BRUCE_V1.4_simplified/meshes/elbow_pitch_link_r.S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
- added link hip_pitch_link_l, mass 0.720628280; collision mesh filename=package://BRUCE_V1.4_simplified/meshes/hip_pitch_link_l.STL; visual mesh filename=package://BRUCE_V1.4_simplified/meshes/hip_pitch_link_l.STL
- added link hip_pitch_link_r, mass 0.728489880; collision mesh filename=package://BRUCE_V1.4_simplified/meshes/hip_pitch_link_r.STL; visual mesh filename=package://BRUCE_V1.4_simplified/meshes/hip_pitch_link_r.STL
- added link hip_roll_link_l, mass 0.003857478; collision mesh filename=package://BRUCE_V1.4_simplified/meshes/hip_roll_link_l.STL; visual mesh filename=package://BRUCE_V1.4_simplified/meshes/hip_roll_link_l.STL
- added link hip_roll_link_r, mass 0.003857478; collision mesh filename=package://BRUCE_V1.4_simplified/meshes/hip_roll_link_r.STL; visual mesh filename=package://BRUCE_V1.4_simplified/meshes/hip_roll_link_r.STL
- added link hip_yaw_link_l, mass 0.637386210; collision mesh filename=package://BRUCE_V1.4_simplified/meshes/hip_yaw_link_l.STL; visual mesh filename=package://BRUCE_V1.4_simplified/meshes/hip_yaw_link_l.STL
- added link hip_yaw_link_r, mass 0.637562640; collision mesh filename=package://BRUCE_V1.4_simplified/meshes/hip_yaw_link_r.STL; visual mesh filename=package://BRUCE_V1.4_simplified/meshes/hip_yaw_link_r.STL
- added link knee_pitch_link_l, mass 0.095265430; collision mesh filename=package://BRUCE_V1.4_simplified/meshes/knee_pitch_link_l.STL; visual mesh filename=package://BRUCE_V1.4_simplified/meshes/knee_pitch_link_l.STL
- added link knee_pitch_link_r, mass 0.095665440; collision mesh filename=package://BRUCE_V1.4_simplified/meshes/knee_pitch_link_r.STL; visual mesh filename=package://BRUCE_V1.4_simplified/meshes/knee_pitch_link_r.STL
- added link shoulder_pitch_link_l, mass 0.049316860; collision mesh filename=package://BRUCE_V1.4_simplified/meshes/shoulder_pitch_link_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; visual mesh filename=package://BRUCE_V1.4_simplified/meshes/shoulder_pitch_link_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
- added link shoulder_pitch_link_r, mass 0.049316860; collision mesh filename=package://BRUCE_V1.4_simplified/meshes/shoulder_pitch_link_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; visual mesh filename=package://BRUCE_V1.4_simplified/meshes/shoulder_pitch_link_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
- added link shoulder_roll_link_l, mass 0.031365250; collision mesh filename=package://BRUCE_V1.4_simplified/meshes/shoulder_roll_link_l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; visual mesh filename=package://BRUCE_V1.4_simplified/meshes/shoulder_roll_link_l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
- added link shoulder_roll_link_r, mass 0.024000000; collision mesh filename=package://BRUCE_V1.4_simplified/meshes/shoulder_roll_link_r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; visual mesh filename=package://BRUCE_V1.4_simplified/meshes/shoulder_roll_link_r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
- link base_link: geometry collision mesh filename=package://BRUCE_V1.4_simplified/meshes/base_link.STL; visual mesh filename=package://BRUCE_V1.4_simplified/meshes/base_link.STL
Joints:
- joint ankle_pitch_l: parent knee_pitch_l -> knee_pitch_link_l
- joint ankle_pitch_r: parent knee_pitch_r -> knee_pitch_link_r
- joint elbow_pitch_l: parent shoulder_roll_l -> shoulder_roll_link_l
- joint elbow_pitch_r: parent shoulder_roll_r -> shoulder_roll_link_r
- joint hip_pitch_l: parent hip_roll_l -> hip_roll_link_l
- joint hip_pitch_r: parent hip_roll_r -> hip_roll_link_r
- joint hip_roll_l: parent hip_yaw_l -> hip_yaw_link_l
- joint hip_roll_r: parent hip_yaw_r -> hip_yaw_link_r
- joint knee_pitch_l: parent hip_pitch_l -> hip_pitch_link_l
- joint knee_pitch_r: parent hip_pitch_r -> hip_pitch_link_r
- joint shoulder_roll_l: parent shoulder_pitch_l -> shoulder_pitch_link_l
- joint shoulder_roll_r: parent shoulder_pitch_r -> shoulder_pitch_link_r
