Commit message: --

File: files/bruce.urdf (robot description, URDF)
Before this commit: robot bruce, 17 links, 16 joints
Links:
- link ankle_pitch_link_l: geometry collision mesh filename=package://bruce/meshes/ankle_pitch_link_l.STL; visual mesh filename=package://bruce/meshes/ankle_pitch_link_l.STL
- link ankle_pitch_link_r: geometry collision mesh filename=package://bruce/meshes/ankle_pitch_link_r.STL; visual mesh filename=package://bruce/meshes/ankle_pitch_link_r.STL
- link base_link: geometry collision mesh filename=package://bruce/meshes/base_link.STL; visual mesh filename=package://bruce/meshes/base_link.STL
- link elbow_pitch_link_l: geometry collision mesh filename=package://bruce/meshes/elbow_pitch_link_l.STL; visual mesh filename=package://bruce/meshes/elbow_pitch_link_l.STL
- link elbow_pitch_link_r: geometry collision mesh filename=package://bruce/meshes/elbow_pitch_link_r.STL; visual mesh filename=package://bruce/meshes/elbow_pitch_link_r.STL
- link hip_pitch_link_l: geometry collision mesh filename=package://bruce/meshes/hip_pitch_link_l.STL; visual mesh filename=package://bruce/meshes/hip_pitch_link_l.STL
- link hip_pitch_link_r: geometry collision mesh filename=package://bruce/meshes/hip_pitch_link_r.STL; visual mesh filename=package://bruce/meshes/hip_pitch_link_r.STL
- link hip_roll_link_l: geometry collision mesh filename=package://bruce/meshes/hip_roll_link_l.STL; visual mesh filename=package://bruce/meshes/hip_roll_link_l.STL
- link hip_roll_link_r: geometry collision mesh filename=package://bruce/meshes/hip_roll_link_r.STL; visual mesh filename=package://bruce/meshes/hip_roll_link_r.STL
- link hip_yaw_link_l: geometry collision mesh filename=package://bruce/meshes/hip_yaw_link_l.STL; visual mesh filename=package://bruce/meshes/hip_yaw_link_l.STL
- link hip_yaw_link_r: geometry collision mesh filename=package://bruce/meshes/hip_yaw_link_r.STL; visual mesh filename=package://bruce/meshes/hip_yaw_link_r.STL
- link knee_pitch_link_l: geometry collision mesh filename=package://bruce/meshes/knee_pitch_link_l.STL; visual mesh filename=package://bruce/meshes/knee_pitch_link_l.STL
- link knee_pitch_link_r: geometry collision mesh filename=package://bruce/meshes/knee_pitch_link_r.STL; visual mesh filename=package://bruce/meshes/knee_pitch_link_r.STL
- link shoulder_pitch_link_l: geometry collision mesh filename=package://bruce/meshes/shoulder_pitch_link_l.STL; visual mesh filename=package://bruce/meshes/shoulder_pitch_link_l.STL
- link shoulder_pitch_link_r: geometry collision mesh filename=package://bruce/meshes/shoulder_pitch_link_r.STL; visual mesh filename=package://bruce/meshes/shoulder_pitch_link_r.STL
- link shoulder_roll_link_l: geometry collision mesh filename=package://bruce/meshes/shoulder_roll_link_l.STL; visual mesh filename=package://bruce/meshes/shoulder_roll_link_l.STL
- link shoulder_roll_link_r: geometry collision mesh filename=package://bruce/meshes/shoulder_roll_link_r.STL; visual mesh filename=package://bruce/meshes/shoulder_roll_link_r.STL

Commit message: update urdf

File: files/bruce.urdf (robot description, URDF)
Before this commit: robot bruce, 17 links, 16 joints
Links:
- link ankle_pitch_link_l: mass 0.027482910 -> 0.02748291
- link ankle_pitch_link_r: mass 0.027626470 -> 0.02762647
- link base_link: mass 1.316889220 -> 1.31688922
- link elbow_pitch_link_l: mass 0.052440370 -> 0.05244037
- link elbow_pitch_link_r: mass 0.052440370 -> 0.05244037
- link hip_pitch_link_l: mass 0.720628280 -> 0.72062828
- link hip_pitch_link_r: mass 0.728489880 -> 0.72848988
- link hip_yaw_link_l: mass 0.637386210 -> 0.63738621
- link hip_yaw_link_r: mass 0.637562640 -> 0.63756264
- link knee_pitch_link_l: mass 0.095265430 -> 0.09526543
- link knee_pitch_link_r: mass 0.095665440 -> 0.09566544
- link shoulder_pitch_link_l: mass 0.049316860 -> 0.04931686
- link shoulder_pitch_link_r: mass 0.049316860 -> 0.04931686
- link shoulder_roll_link_l: mass 0.031365250 -> 0.03136525
- link shoulder_roll_link_r: mass 0.024000000 -> 0.024
Joints:
- joint elbow_pitch_l: limit lower=1 upper=1 effort=1 velocity=1 -> lower=0 upper=0 effort=0 velocity=0
- joint hip_pitch_r: limit lower=1 upper=1 effort=1 velocity=1 -> lower=0 upper=0 effort=0 velocity=0
- joint hip_roll_l: axis 0 0 -1 -> 0 0 1; origin xyz=0 0 0 rpy=1.570796327 1.570796327 0 -> xyz=0 0 0 rpy=1.570796327 1.570796327 3.14159
- joint hip_roll_r: axis 0 0 -1 -> 0 0 1; origin xyz=0 0 0 rpy=1.570796327 1.570796327 0 -> xyz=0 0 0 rpy=-1.570796327 1.570796327 0
- joint hip_yaw_r: limit lower=1 upper=1 effort=1 velocity=1 -> lower=0 upper=0 effort=0 velocity=0
- joint knee_pitch_r: axis 0 0 -1 -> 0 0 1
- joint shoulder_pitch_l: origin xyz=0.029216 0.12375 0.152985 rpy=1.570796327 -1.570796327 0 -> xyz=0.029216 0.12375 0.152985 rpy=-1.570796327 1.570796327 0
